File: Synapse RPi3 Adapter/Rev A/synapse_rpi3_adapter.sch (EAGLE design)
At the start: 3 parts, among them J1 PPTC202LFBN-RC, J2 NPPN121BFCN-RC, J3 NPPN121BFCN-RC

Commit message: Synapse RPi3 Adapter Schematic 2
Parts:
- added C1: 100nF, rcl:C-EUC0603
- added C2: (no value), rcl:C-EUC0603
- added D1, D2: WP130WDT/EGW, KVB-ICs:WP130WDT/EGW
- added FD1, FD2: FIDUCIALUFIDUCIAL, KVB-misc:FIDUCIALUFIDUCIAL
- added MNT1, MNT2: MOUNT-HOLE-NO-PLATE5.0MM, KVB-misc:MOUNT-HOLE-NO-PLATE5.0MM
- added MNT3, MNT4: MOUNT-HOLE-NO-PLATE320MILS, KVB-misc:MOUNT-HOLE-NO-PLATE320MILS
- added R1, R2, R3, R4: 68.1, rcl:R-US_R0603
- added R5, R6: 10.0K, rcl:R-US_R0603
- added S1: 1-1825027-7, KVB-switches:1-1825027-7
- added TP1, TP2, TP3: TEST-POINT, KVB-misc:TEST-POINT
Connections:
- new net !SNPS_RESET: C2.1, J3.P$11, R6.1
- new net N$1: D1.RED, R1.1
- new net N$2: D1.GRN, R2.1
- new net N$3: D2.RED, R3.1
- new net N$4: D2.GRN, R4.1
- new net RPI3_GREEN: J1.29, R4.2
- new net RPI3_RED: J1.31, R3.2
- new net RPI3_SW: C1.1, J1.37, R5.1, S1.P$2
- new net SNPS_GREEN: J2.P$3, R2.2
- new net SNPS_RED: J2.P$2, R1.2
- net 0V: now also C1.2, C2.2, D1.P$2, D2.P$2, S1.GND1, S1.GND2, S1.P$1, TP3.PP
- net 3.3V: now also R5.2, R6.2, TP1.PP
- net 5.0V: now also TP2.PP
Other:
- note added: "(2Vf, 20mA x 4)"
- note added: "LEDs"
- note added: "Misc"
- note added: "RPi3 Switch"
- note added: "Supply Test Points"
- note added: "Synapse Reset"
- moved on the sheet: J3

Commit message: Synapse RPi3 Layout 1
Parts:
- removed MNT3, MNT4: MOUNT-HOLE-NO-PLATE320MILS, KVB-misc:MOUNT-HOLE-NO-PLATE320MILS
- added U$1: BA_LOGO, KVB-misc:BA_LOGO
- added X1: RF200PD1, KVB-misc:RF200PD1
- C2: value (none) -> 10nF
Other:
- moved on the sheet: TP1, TP2, TP3
