File: Synapse RPi3 Adapter/Rev B/synapse_rpi3_adapter.brd (EAGLE design)
At the start: 56 x 65 mm, 24 parts, among them J1 PPTC202LFBN-RC, J2 NPPN121BFCN-RC, J3 NPPN121BFCN-RC, X1 RF200PD1

Commit message: Synapse RPi3 Rev. B 2
Connections:
- net UART_RX: now also J2.10; no longer J2.5
- net UART_TX: now also J2.9; no longer J2.6
Routing:
- net UART_TX: track 12.8 -> 17.8 mm
- net UART_RX: track 16.5 -> 17.3 mm
Changed lines of the file:
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@@
 <grid distance="50" unitdist="mil" unit="mil" style="lines" multiple="1" display="yes" altdistance="25" altunitdist="mil" altunit="mil"/>
 <layers>
-<layer number="1" name="Top" color="4" fill="1" visible="yes" active="yes"/>
+<layer number="1" name="Top" color="4" fill="1" visible="no" active="yes"/>
 <layer number="2" name="Route2" color="1" fill="3" visible="no" active="no"/>
 <layer number="3" name="Route3" color="4" fill="3" visible="no" active="no"/>
@@
 <layer number="14" name="Route14" color="1" fill="6" visible="no" active="no"/>
 <layer number="15" name="Route15" color="4" fill="6" visible="no" active="no"/>
-<layer number="16" name="Bottom" color="1" fill="1" visible="no" active="yes"/>
+<layer number="16" name="Bottom" color="1" fill="1" visible="yes" active="yes"/>
 <layer number="17" name="Pads" color="2" fill="1" visible="yes" active="yes"/>
 <layer number="18" name="Vias" color="2" fill="1" visible="yes" active="yes"/>
 <layer number="19" name="Unrouted" color="6" fill="1" visible="yes" active="yes"/>
 <layer number="20" name="Dimension" color="15" fill="1" visible="yes" active="yes"/>
-<layer number="21" name="tPlace" color="7" fill="1" visible="yes" active="yes"/>
-<layer number="22" name="bPlace" color="7" fill="1" visible="no" active="yes"/>
-<layer number="23" name="tOrigins" color="15" fill="1" visible="yes" active="yes"/>
-<layer number="24" name="bOrigins" color="15" fill="1" visible="no" active="yes"/>
-<layer number="25" name="tNames" color="7" fill="1" visible="yes" active="yes"/>
-<layer number="26" name="bNames" color="7" fill="1" visible="no" active="yes"/>
+<layer number="21" name="tPlace" color="7" fill="1" visible="no" active="yes"/>
+<layer number="22" name="bPlace" color="7" fill="1" visible="yes" active="yes"/>
+<layer number="23" name="tOrigins" color="15" fill="1" visible="no" active="yes"/>
+<layer number="24" name="bOrigins" color="15" fill="1" visible="yes" active="yes"/>
+<layer number="25" name="tNames" color="7" fill="1" visible="no" active="yes"/>
+<layer number="26" name="bNames" color="7" fill="1" visible="yes" active="yes"/>
 <layer number="27" name="tValues" color="7" fill="1" visible="no" active="yes"/>
 <layer number="28" name="bValues" color="7" fill="1" visible="no" active="yes"/>
@@
 <layer number="49" name="Reference" color="7" fill="1" visible="yes" active="yes"/>
 <layer number="50" name="dxf" color="7" fill="1" visible="no" active="no"/>
-<layer number="51" name="tDocu" color="7" fill="1" visible="yes" active="yes"/>
-<layer number="52" name="bDocu" color="7" fill="1" visible="no" active="yes"/>
+<layer number="51" name="tDocu" color="7" fill="1" visible="no" active="yes"/>
+<layer number="52" name="bDocu" color="7" fill="1" visible="yes" active="yes"/>
 <layer number="53" name="tGND_GNDA" color="7" fill="9" visible="no" active="no"/>
 <layer number="54" name="bGND_GNDA" color="1" fill="9" visible="no" active="no"/>
@@
 <signal name="UART_TX">
 <contactref element="J1" pad="8"/>
-<contactref element="J2" pad="6"/>
 <wire x1="52.512" y1="47.752" x2="53.77" y2="49.01" width="0.2032" layer="16"/>
-<wire x1="52.512" y1="47.752" x2="48.657" y2="47.752" width="0.2032" layer="16"/>
-<wire x1="48.657" y1="47.752" x2="43.5864" y2="42.6814" width="0.2032" layer="16"/>
+<wire x1="52.512" y1="47.752" x2="50.292" y2="47.752" width="0.2032" layer="16"/>
+<contactref element="J2" pad="9"/>
+<wire x1="43.5864" y1="36.6814" x2="46.99" y2="40.085" width="0.2032" layer="16"/>
+<wire x1="46.99" y1="40.085" x2="46.99" y2="44.45" width="0.2032" layer="16"/>
+<wire x1="46.99" y1="44.45" x2="50.292" y2="47.752" width="0.2032" layer="16"/>
 </signal>
 <signal name="UART_RX">
 <contactref element="J1" pad="10"/>
-<contactref element="J2" pad="5"/>
-<wire x1="48.514" y1="45.085" x2="52.385" y2="45.085" width="0.2032" layer="16"/>
+<wire x1="50.165" y1="45.085" x2="52.385" y2="45.085" width="0.2032" layer="16"/>
 <wire x1="52.385" y1="45.085" x2="53.77" y2="46.47" width="0.2032" layer="16"/>
-<wire x1="48.514" y1="45.085" x2="45.085" y2="41.656" width="0.2032" layer="16"/>
-<wire x1="45.085" y1="41.656" x2="42.799" y2="41.656" width="0.2032" layer="16"/>
-<wire x1="42.799" y1="41.656" x2="42.545" y2="41.91" width="0.2032" layer="16"/>
-<wire x1="42.545" y1="41.91" x2="42.545" y2="43.64" width="0.2032" layer="16"/>
-<wire x1="42.545" y1="43.64" x2="43.5864" y2="44.6814" width="0.2032" layer="16"/>
+<contactref element="J2" pad="10"/>
+<wire x1="43.5864" y1="34.6814" x2="48.26" y2="39.355" width="0.2032" layer="16"/>
+<wire x1="48.26" y1="39.355" x2="48.26" y2="43.18" width="0.2032" layer="16"/>
+<wire x1="48.26" y1="43.18" x2="50.165" y2="45.085" width="0.2032" layer="16"/>
 </signal>
 <signal name="N$1">

Commit message: Synapse RPi3 Rev. B 3
Connections:
- net SNPS_GREEN: now also J2.2; no longer J2.3
- net SNPS_RED: now also J2.3; no longer J2.2
Routing:
- net SNPS_RED: track 35.8 -> 29.4 mm
- net SNPS_GREEN: track 25.3 -> 23.5 mm
Changed lines of the file:
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@@
 <grid distance="50" unitdist="mil" unit="mil" style="lines" multiple="1" display="yes" altdistance="25" altunitdist="mil" altunit="mil"/>
 <layers>
-<layer number="1" name="Top" color="4" fill="1" visible="no" active="yes"/>
+<layer number="1" name="Top" color="4" fill="1" visible="yes" active="yes"/>
 <layer number="2" name="Route2" color="1" fill="3" visible="no" active="no"/>
 <layer number="3" name="Route3" color="4" fill="3" visible="no" active="no"/>
@@
 </signal>
 <signal name="SNPS_RED">
+<contactref element="R1" pad="2"/>
+<contactref element="J2" pad="3"/>
+<wire x1="43.5864" y1="48.6814" x2="22.2236" y2="48.6814" width="0.2032" layer="1"/>
+<wire x1="22.2236" y1="48.6814" x2="16.51" y2="54.395" width="0.2032" layer="1"/>
+</signal>
+<signal name="SNPS_GREEN">
+<contactref element="R2" pad="2"/>
 <contactref element="J2" pad="2"/>
-<contactref element="R1" pad="2"/>
-<wire x1="16.51" y1="52.832" x2="16.51" y2="54.395" width="0.2032" layer="1"/>
-<wire x1="43.5864" y1="50.6814" x2="43.9336" y2="50.6814" width="0.2032" layer="1"/>
-<wire x1="43.9336" y1="50.6814" x2="45.085" y2="49.53" width="0.2032" layer="1"/>
-<wire x1="45.085" y1="49.53" x2="45.085" y2="48.26" width="0.2032" layer="1"/>
-<wire x1="45.085" y1="48.26" x2="44.5135" y2="47.6885" width="0.2032" layer="1"/>
-<wire x1="44.5135" y1="47.6885" x2="21.6535" y2="47.6885" width="0.2032" layer="1"/>
-<wire x1="21.6535" y1="47.6885" x2="16.51" y2="52.832" width="0.2032" layer="1"/>
-</signal>
-<signal name="SNPS_GREEN">
-<contactref element="J2" pad="3"/>
-<contactref element="R2" pad="2"/>
-<wire x1="21.59" y1="52.832" x2="21.59" y2="54.395" width="0.2032" layer="1"/>
-<wire x1="43.5864" y1="48.6814" x2="25.7406" y2="48.6814" width="0.2032" layer="1"/>
-<wire x1="25.7406" y1="48.6814" x2="21.59" y2="52.832" width="0.2032" layer="1"/>
+<wire x1="43.5864" y1="50.6814" x2="25.3036" y2="50.6814" width="0.2032" layer="1"/>
+<wire x1="25.3036" y1="50.6814" x2="21.59" y2="54.395" width="0.2032" layer="1"/>
 </signal>
 <signal name="RPI3_GREEN">
