File: Synapse RPi3 Adapter/Rev B/synapse_rpi3_adapter.sch (EAGLE design)
At the start: 24 parts, among them J1 PPTC202LFBN-RC, J2 NPPN121BFCN-RC, J3 NPPN121BFCN-RC, X1 RF200PD1

Commit message: Synapse RPi3 Rev. B 2
Connections:
- net UART_RX: now also J2.P$10; no longer J2.P$5
- net UART_TX: now also J2.P$9; no longer J2.P$6
Changed lines of the file:
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@@
 </segment>
 <segment>
-<pinref part="J2" gate="G$1" pin="P$6"/>
-<wire x1="40.64" y1="142.24" x2="33.02" y2="142.24" width="0.1524" layer="91"/>
-<label x="20.32" y="142.24" size="1.778" layer="95"/>
+<pinref part="J2" gate="G$1" pin="P$9"/>
+<wire x1="40.64" y1="134.62" x2="33.02" y2="134.62" width="0.1524" layer="91"/>
+<label x="20.32" y="134.62" size="1.778" layer="95"/>
 </segment>
 </net>
@@
 </segment>
 <segment>
-<pinref part="J2" gate="G$1" pin="P$5"/>
-<wire x1="40.64" y1="144.78" x2="33.02" y2="144.78" width="0.1524" layer="91"/>
-<label x="20.32" y="144.78" size="1.778" layer="95"/>
+<pinref part="J2" gate="G$1" pin="P$10"/>
+<wire x1="40.64" y1="132.08" x2="33.02" y2="132.08" width="0.1524" layer="91"/>
+<label x="20.32" y="132.08" size="1.778" layer="95"/>
 </segment>
 </net>

Commit message: Synapse RPi3 Rev. B 3
Connections:
- net SNPS_GREEN: now also J2.P$2; no longer J2.P$3
- net SNPS_RED: now also J2.P$3; no longer J2.P$2
Changed lines of the file:
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@@
 <net name="SNPS_RED" class="0">
-<segment>
-<pinref part="J2" gate="G$1" pin="P$2"/>
-<wire x1="40.64" y1="152.4" x2="33.02" y2="152.4" width="0.1524" layer="91"/>
-<label x="15.24" y="152.4" size="1.778" layer="95"/>
-</segment>
 <segment>
 <pinref part="R1" gate="G$1" pin="2"/>
@@
 <label x="7.62" y="78.74" size="1.778" layer="95"/>
 </segment>
-</net>
-<net name="SNPS_GREEN" class="0">
 <segment>
 <pinref part="J2" gate="G$1" pin="P$3"/>
@@
 <label x="15.24" y="149.86" size="1.778" layer="95"/>
 </segment>
+</net>
+<net name="SNPS_GREEN" class="0">
 <segment>
 <pinref part="R2" gate="G$1" pin="2"/>
@@
 <label x="7.62" y="81.28" size="1.778" layer="95"/>
 </segment>
+<segment>
+<pinref part="J2" gate="G$1" pin="P$2"/>
+<wire x1="40.64" y1="152.4" x2="33.02" y2="152.4" width="0.1524" layer="91"/>
+<label x="15.24" y="152.4" size="1.778" layer="95"/>
+</segment>
 </net>
